File: hardware/peripheral/p2xgr-001.brd (EAGLE design)
At the start: 18 x 23 mm, 7 parts

Commit message: Clean up.
Parts:
- removed J21, J22, J23, J24: (no value), SparkFun-Connectors:JST-4-PTH-VERT
Connections:
- net ANLG0: no longer J21.2
- net ANLG1: no longer J22.2
- net ANLG2: no longer J23.2
- net ANLG3: no longer J24.2
- net DTCT0: no longer J21.1
- net DTCT1: no longer J22.1
- net DTCT2: no longer J23.1
- net DTCT3: no longer J24.1
- net GND: no longer J21.4, J22.4, J23.4, J24.4
- net VCC: no longer J21.3, J22.3, J23.3, J24.3
Routing:
- net VCC: track 42.2 -> 26.4 mm
- net GND: track 31.1 -> 30.3 mm

Commit message: First working model.
Parts:
- added S1C, S2R: (no value), switch-dil:A1353HEX
- moved U$1 17.0 mm to (17.5, 11.5), turned to 270 degrees
- moved LOGO1 5.39 mm to (5.00, 6.00)
Connections:
- net ANLG0: now also S2R.1
- net ANLG1: now also S2R.4
- net ANLG2: now also S2R.8
- net ANLG3: now also S2R.2
- net DTCT0: now also S1C.1
- net DTCT1: now also S1C.4
- net DTCT2: now also S1C.8
- net DTCT3: now also S1C.2
- net GND: now also S1C.C
- net VCC: now also S2R.C
Routing:
- net ANLG3: track 8.18 -> 15.1 mm
- net DTCT0: track 13.0 -> 17.4 mm
- net ANLG1: track 8.23 -> 12.6 mm
- net GND: track 30.3 -> 26.1 mm
- net ANLG0: track 8.25 -> 5.41 mm
- net DTCT3: track 13.2 -> 15.8 mm
- net DTCT2: track 13.7 -> 11.1 mm
- net VCC: track 26.4 -> 28.4 mm
- net DTCT1: track 13.2 -> 15.0 mm
- net ANLG2: track 8.20 -> 7.26 mm
Other:
- board text removed: "0"
- board text removed: "A"
- board text removed: "D"
- board text removed: "G"
- board text removed: "V"
