File: hardware/peripheral/p2xgr-001.sch (EAGLE design)
At the start: 7 parts

Commit message: Clean up.
Parts:
- removed J21, J22, J23, J24: (no value), SparkFun-Connectors:CONN_04JST-PTH-VERT
Connections:
- net ANLG0: no longer J21.2
- net ANLG1: no longer J22.2
- net ANLG2: no longer J23.2
- net ANLG3: no longer J24.2
- net DTCT0: no longer J21.1
- net DTCT1: no longer J22.1
- net DTCT2: no longer J23.1
- net DTCT3: no longer J24.1
- net GND: no longer J21.4, J22.4, J23.4, J24.4
- net VCC: no longer J21.3, J22.3, J23.3, J24.3
Changed lines of the file:
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@@
 <part name="SUPPLY3" library="supply2" library_urn="urn:adsk.eagle:library:372" deviceset="VCC" device=""/>
 <part name="U$1" library="pineapple" deviceset="PINEAPPLE450_SILK" device=""/>
-<part name="J21" library="SparkFun-Connectors" library_urn="urn:adsk.eagle:library:513" deviceset="CONN_04" device="JST-PTH-VERT" package3d_urn="urn:adsk.eagle:package:38102/1"/>
-<part name="J22" library="SparkFun-Connectors" library_urn="urn:adsk.eagle:library:513" deviceset="CONN_04" device="JST-PTH-VERT" package3d_urn="urn:adsk.eagle:package:38102/1"/>
-<part name="J23" library="SparkFun-Connectors" library_urn="urn:adsk.eagle:library:513" deviceset="CONN_04" device="JST-PTH-VERT" package3d_urn="urn:adsk.eagle:package:38102/1"/>
-<part name="J24" library="SparkFun-Connectors" library_urn="urn:adsk.eagle:library:513" deviceset="CONN_04" device="JST-PTH-VERT" package3d_urn="urn:adsk.eagle:package:38102/1"/>
 </parts>
 <sheets>
@@
 </instance>
 <instance part="U$1" gate="G$1" x="241.3" y="142.24" smashed="yes"/>
-<instance part="J21" gate="G$1" x="48.26" y="121.92" smashed="yes">
-<attribute name="VALUE" x="43.18" y="114.554" size="1.778" layer="96" font="vector"/>
-<attribute name="NAME" x="43.18" y="130.048" size="1.778" layer="95" font="vector"/>
-</instance>
-<instance part="J22" gate="G$1" x="48.26" y="104.14" smashed="yes">
-<attribute name="VALUE" x="43.18" y="96.774" size="1.778" layer="96" font="vector"/>
-<attribute name="NAME" x="43.18" y="112.268" size="1.778" layer="95" font="vector"/>
-</instance>
-<instance part="J23" gate="G$1" x="48.26" y="86.36" smashed="yes">
-<attribute name="VALUE" x="43.18" y="78.994" size="1.778" layer="96" font="vector"/>
-<attribute name="NAME" x="43.18" y="94.488" size="1.778" layer="95" font="vector"/>
-</instance>
-<instance part="J24" gate="G$1" x="48.26" y="68.58" smashed="yes">
-<attribute name="VALUE" x="43.18" y="61.214" size="1.778" layer="96" font="vector"/>
-<attribute name="NAME" x="43.18" y="76.708" size="1.778" layer="95" font="vector"/>
-</instance>
 </instances>
 <busses>
@@
 <junction x="101.6" y="93.98"/>
 </segment>
-<segment>
-<pinref part="J21" gate="G$1" pin="4"/>
-<wire x1="53.34" y1="127" x2="58.42" y2="127" width="0.1524" layer="91"/>
-<label x="58.42" y="127" size="0.8128" layer="95" xref="yes"/>
-</segment>
-<segment>
-<pinref part="J22" gate="G$1" pin="4"/>
-<wire x1="53.34" y1="109.22" x2="58.42" y2="109.22" width="0.1524" layer="91"/>
-<label x="58.42" y="109.22" size="0.8128" layer="95" xref="yes"/>
-</segment>
-<segment>
-<pinref part="J23" gate="G$1" pin="4"/>
-<wire x1="53.34" y1="91.44" x2="58.42" y2="91.44" width="0.1524" layer="91"/>
-<label x="58.42" y="91.44" size="0.8128" layer="95" xref="yes"/>
-</segment>
-<segment>
-<pinref part="J24" gate="G$1" pin="4"/>
-<wire x1="53.34" y1="73.66" x2="58.42" y2="73.66" width="0.1524" layer="91"/>
-<label x="58.42" y="73.66" size="0.8128" layer="95" xref="yes"/>
-</segment>
 </net>
 <net name="DTCT0" class="0">
@@
 <wire x1="116.84" y1="109.22" x2="132.08" y2="109.22" width="0.1524" layer="91"/>
 <label x="132.08" y="109.22" size="0.8128" layer="95" xref="yes"/>
-</segment>
-<segment>
-<pinref part="J21" gate="G$1" pin="1"/>
-<wire x1="53.34" y1="119.38" x2="58.42" y2="119.38" width="0.1524" layer="91"/>
-<label x="58.42" y="119.38" size="0.8128" layer="95" xref="yes"/>
 </segment>
 </net>
@@
 <junction x="124.46" y="101.6"/>
 </segment>
-<segment>
-<pinref part="J21" gate="G$1" pin="3"/>
-<wire x1="53.34" y1="124.46" x2="58.42" y2="124.46" width="0.1524" layer="91"/>
-<label x="58.42" y="124.46" size="0.8128" layer="95" xref="yes"/>
-</segment>
-<segment>
-<pinref part="J22" gate="G$1" pin="3"/>
-<wire x1="53.34" y1="106.68" x2="58.42" y2="106.68" width="0.1524" layer="91"/>
-<label x="58.42" y="106.68" size="0.8128" layer="95" xref="yes"/>
-</segment>
-<segment>
-<pinref part="J23" gate="G$1" pin="3"/>
-<wire x1="53.34" y1="88.9" x2="58.42" y2="88.9" width="0.1524" layer="91"/>
-<label x="58.42" y="88.9" size="0.8128" layer="95" xref="yes"/>
-</segment>
-<segment>
-<pinref part="J24" gate="G$1" pin="3"/>
-<wire x1="53.34" y1="71.12" x2="58.42" y2="71.12" width="0.1524" layer="91"/>
-<label x="58.42" y="71.12" size="0.8128" layer="95" xref="yes"/>
-</segment>
 </net>
 <net name="DTCT1" class="0">
@@
 <wire x1="116.84" y1="104.14" x2="132.08" y2="104.14" width="0.1524" layer="91"/>
 <label x="132.08" y="104.14" size="0.8128" layer="95" xref="yes"/>
-</segment>
-<segment>
-<pinref part="J22" gate="G$1" pin="1"/>
-<wire x1="53.34" y1="101.6" x2="58.42" y2="101.6" width="0.1524" layer="91"/>
-<label x="58.42" y="101.6" size="0.8128" layer="95" xref="yes"/>
 </segment>
 </net>
@@
 <label x="132.08" y="99.06" size="0.8128" layer="95" xref="yes"/>
 </segment>
-<segment>
-<pinref part="J23" gate="G$1" pin="1"/>
-<wire x1="53.34" y1="83.82" x2="58.42" y2="83.82" width="0.1524" layer="91"/>
-<label x="58.42" y="83.82" size="0.8128" layer="95" xref="yes"/>
-</segment>
 </net>
 <net name="DTCT3" class="0">
@@
 <wire x1="116.84" y1="93.98" x2="132.08" y2="93.98" width="0.1524" layer="91"/>
 <label x="132.08" y="93.98" size="0.8128" layer="95" xref="yes"/>
-</segment>
-<segment>
-<pinref part="J24" gate="G$1" pin="1"/>
-<wire x1="53.34" y1="66.04" x2="58.42" y2="66.04" width="0.1524" layer="91"/>
-<label x="58.42" y="66.04" size="0.8128" layer="95" xref="yes"/>
 </segment>
 </net>
@@
 <label x="96.52" y="106.68" size="0.8128" layer="95" rot="R180" xref="yes"/>
 </segment>
-<segment>
-<pinref part="J21" gate="G$1" pin="2"/>
-<wire x1="53.34" y1="121.92" x2="58.42" y2="121.92" width="0.1524" layer="91"/>
-<label x="58.42" y="121.92" size="0.8128" layer="95" xref="yes"/>
-</segment>
 </net>
 <net name="ANLG1" class="0">
@@
 <wire x1="109.22" y1="101.6" x2="96.52" y2="101.6" width="0.1524" layer="91"/>
 <label x="96.52" y="101.6" size="0.8128" layer="95" rot="R180" xref="yes"/>
-</segment>
-<segment>
-<pinref part="J22" gate="G$1" pin="2"/>
-<wire x1="53.34" y1="104.14" x2="58.42" y2="104.14" width="0.1524" layer="91"/>
-<label x="58.42" y="104.14" size="0.8128" layer="95" xref="yes"/>
 </segment>
 </net>
@@
 <label x="96.52" y="91.44" size="0.8128" layer="95" rot="R180" xref="yes"/>
 </segment>
-<segment>
-<pinref part="J24" gate="G$1" pin="2"/>
-<wire x1="53.34" y1="68.58" x2="58.42" y2="68.58" width="0.1524" layer="91"/>
-<label x="58.42" y="68.58" size="0.8128" layer="95" xref="yes"/>
-</segment>
 </net>
 <net name="ANLG2" class="0">
@@
 <label x="96.52" y="96.52" size="0.8128" layer="95" rot="R180" xref="yes"/>
 </segment>
-<segment>
-<pinref part="J23" gate="G$1" pin="2"/>
-<wire x1="53.34" y1="86.36" x2="58.42" y2="86.36" width="0.1524" layer="91"/>
-<label x="58.42" y="86.36" size="0.8128" layer="95" xref="yes"/>
-</segment>
 </net>

Commit message: First working model.
Parts:
- added S1C, S2R: (no value), switch-dil:A1353HEX
Connections:
- net ANLG0: now also S2R.1
- net ANLG1: now also S2R.4
- net ANLG2: now also S2R.8
- net ANLG3: now also S2R.2
- net DTCT0: now also S1C.1
- net DTCT1: now also S1C.4
- net DTCT2: now also S1C.8
- net DTCT3: now also S1C.2
- net GND: now also S1C.C
- net VCC: now also S2R.C
Changed lines of the file:
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@@
 <part name="SUPPLY3" library="supply2" library_urn="urn:adsk.eagle:library:372" deviceset="VCC" device=""/>
 <part name="U$1" library="pineapple" deviceset="PINEAPPLE450_SILK" device=""/>
+<part name="S1C" library="switch-dil" library_urn="urn:adsk.eagle:library:375" deviceset="A1353HEX" device="" package3d_urn="urn:adsk.eagle:package:27207/1"/>
+<part name="S2R" library="switch-dil" library_urn="urn:adsk.eagle:library:375" deviceset="A1353HEX" device="" package3d_urn="urn:adsk.eagle:package:27207/1"/>
+<part name="SUPPLY2" library="supply2" library_urn="urn:adsk.eagle:library:372" deviceset="GND" device=""/>
+<part name="SUPPLY4" library="supply2" library_urn="urn:adsk.eagle:library:372" deviceset="VCC" device=""/>
 </parts>
 <sheets>
@@
 </instance>
 <instance part="U$1" gate="G$1" x="241.3" y="142.24" smashed="yes"/>
+<instance part="S1C" gate="1" x="40.64" y="99.06" smashed="yes">
+<attribute name="NAME" x="36.195" y="93.98" size="1.778" layer="95" rot="R90"/>
+<attribute name="VALUE" x="49.53" y="93.98" size="1.778" layer="96" rot="R90"/>
+</instance>
+<instance part="S2R" gate="1" x="66.04" y="99.06" smashed="yes" rot="R180">
+<attribute name="NAME" x="70.485" y="104.14" size="1.778" layer="95" rot="R270"/>
+<attribute name="VALUE" x="57.15" y="104.14" size="1.778" layer="96" rot="R270"/>
+</instance>
+<instance part="SUPPLY2" gate="GND" x="40.64" y="76.2" smashed="yes">
+<attribute name="VALUE" x="38.735" y="73.025" size="1.778" layer="96"/>
+</instance>
+<instance part="SUPPLY4" gate="G$1" x="66.04" y="116.84" smashed="yes">
+<attribute name="VALUE" x="64.135" y="120.015" size="1.778" layer="96"/>
+</instance>
 </instances>
 <busses>
@@
 <junction x="101.6" y="93.98"/>
 </segment>
+<segment>
+<pinref part="S1C" gate="1" pin="C"/>
+<wire x1="40.64" y1="91.44" x2="40.64" y2="78.74" width="0.1524" layer="91"/>
+<pinref part="SUPPLY2" gate="GND" pin="GND"/>
+</segment>
 </net>
 <net name="DTCT0" class="0">
@@
 <wire x1="116.84" y1="109.22" x2="132.08" y2="109.22" width="0.1524" layer="91"/>
 <label x="132.08" y="109.22" size="0.8128" layer="95" xref="yes"/>
+</segment>
+<segment>
+<pinref part="S1C" gate="1" pin="1"/>
+<wire x1="38.1" y1="106.68" x2="38.1" y2="114.3" width="0.1524" layer="91"/>
+<label x="38.1" y="114.3" size="0.8128" layer="95" rot="R90" xref="yes"/>
 </segment>
 </net>
@@
 <junction x="124.46" y="101.6"/>
 </segment>
+<segment>
+<pinref part="S2R" gate="1" pin="C"/>
+<wire x1="66.04" y1="106.68" x2="66.04" y2="114.3" width="0.1524" layer="91"/>
+<pinref part="SUPPLY4" gate="G$1" pin="VCC"/>
+</segment>
 </net>
 <net name="DTCT1" class="0">
@@
 <label x="132.08" y="104.14" size="0.8128" layer="95" xref="yes"/>
 </segment>
+<segment>
+<pinref part="S1C" gate="1" pin="4"/>
+<wire x1="43.18" y1="106.68" x2="43.18" y2="114.3" width="0.1524" layer="91"/>
+<label x="43.18" y="114.3" size="0.8128" layer="95" rot="R90" xref="yes"/>
+</segment>
 </net>
 <net name="DTCT2" class="0">
@@
 <label x="132.08" y="99.06" size="0.8128" layer="95" xref="yes"/>
 </segment>
+<segment>
+<pinref part="S1C" gate="1" pin="8"/>
+<wire x1="45.72" y1="106.68" x2="45.72" y2="114.3" width="0.1524" layer="91"/>
+<label x="45.72" y="114.3" size="0.8128" layer="95" rot="R90" xref="yes"/>
+</segment>
 </net>
 <net name="DTCT3" class="0">
@@
 <label x="132.08" y="93.98" size="0.8128" layer="95" xref="yes"/>
 </segment>
+<segment>
+<pinref part="S1C" gate="1" pin="2"/>
+<wire x1="40.64" y1="106.68" x2="40.64" y2="114.3" width="0.1524" layer="91"/>
+<label x="40.64" y="114.3" size="0.8128" layer="95" rot="R90" xref="yes"/>
+</segment>
 </net>
 <net name="ANLG0" class="0">
@@
 <label x="96.52" y="106.68" size="0.8128" layer="95" rot="R180" xref="yes"/>
 </segment>
+<segment>
+<pinref part="S2R" gate="1" pin="1"/>
+<wire x1="68.58" y1="91.44" x2="68.58" y2="86.36" width="0.1524" layer="91"/>
+<label x="68.58" y="86.36" size="0.8128" layer="95" rot="R270" xref="yes"/>
+</segment>
 </net>
 <net name="ANLG1" class="0">
@@
 <label x="96.52" y="101.6" size="0.8128" layer="95" rot="R180" xref="yes"/>
 </segment>
+<segment>
+<pinref part="S2R" gate="1" pin="4"/>
+<wire x1="63.5" y1="91.44" x2="63.5" y2="86.36" width="0.1524" layer="91"/>
+<label x="63.5" y="86.36" size="0.8128" layer="95" rot="R270" xref="yes"/>
+</segment>
 </net>
 <net name="ANLG3" class="0">
@@
 <label x="96.52" y="91.44" size="0.8128" layer="95" rot="R180" xref="yes"/>
 </segment>
+<segment>
+<pinref part="S2R" gate="1" pin="2"/>
+<wire x1="66.04" y1="91.44" x2="66.04" y2="86.36" width="0.1524" layer="91"/>
+<label x="66.04" y="86.36" size="0.8128" layer="95" rot="R270" xref="yes"/>
+</segment>
 </net>
 <net name="ANLG2" class="0">
@@
 <label x="96.52" y="96.52" size="0.8128" layer="95" rot="R180" xref="yes"/>
 </segment>
-</net>
+<segment>
+<pinref part="S2R" gate="1" pin="8"/>
+<wire x1="60.96" y1="91.44" x2="60.96" y2="86.36" width="0.1524" layer="91"/>
+<label x="60.96" y="86.36" size="0.8128" layer="95" rot="R270" xref="yes"/>
+</segment>
+</net>
